Commit message: Localization seems to work properly in rviz now

File: src/robot_description/description/robot_description.urdf (robot description, URDF)
Before this commit: robot robot, 2 links, 1 joints
Links:
- removed link base_footprint
- added link gps
- added link laser
Joints:
- removed joint base_joint
- added joint gps_joint: type fixed, parent base_link, child gps, origin xyz=${12 * inches} 0 ${8 * inches} rpy=0 0 0
- added joint laser_joint: type fixed, parent base_link, child laser, origin xyz=${12 * inches} 0 ${8 * inches} rpy=0 0 ${pi}
