Commit message: Added the base footprint link to the urdf

File: src/robot_bringup/urdf/robot_description.urdf (robot description, URDF)
Before this commit: robot robot, 3 links, 2 joints
Links:
- added link base_footprint
Joints:
- added joint base_joint: type fixed, parent base_link, child base_footprint, origin xyz=0 0 0 rpy=0 0 0

Commit message: Updated URDF

File: src/robot_bringup/urdf/robot_description.urdf (robot description, URDF)
Before this commit: robot robot, 4 links, 3 joints
Joints:
- joint gps_joint: origin xyz=${12 * inches} 0 ${8 * inches} rpy=0 0 0 -> xyz=0 0 ${8 * inches} rpy=0 0 0
- joint laser_joint: origin xyz=${12 * inches} 0 ${8 * inches} rpy=0 0 ${pi} -> xyz=0 0 ${8 * inches} rpy=0 0 ${pi}
